File: pcb/kicad/left/left.kicad_pcb (KiCad board)
At the start: 2 copper layers, 135.9 x 89.9 mm, 61 parts, among them J1 USB_C_Receptacle_USB2.0, J2 AudioJack4, J3 Conn_01x12_Male, SW1 BOOT, SW10 SW_Push, SW12 SW_Push, SW13 SW_Push, SW14 SW_Push, SW15 SW_Push, SW17 SW_Push, SW18 SW_Push, SW19 SW_Push, SW2 RESET, SW21 SW_Push, SW22 SW_Push, SW23 SW_Push, SW24 SW_Push, SW3 SW_Push, SW31 SW_Push, SW32 SW_Push, SW33 SW_Push, SW34 SW_Push, SW4 SW_Push, SW5 SW_Push, SW7 SW_Push, SW8 SW_Push, SW9 SW_Push, U1 STM32, U2 LDO

Commit message: yeet.
Parts:
- removed D17: D4.6, Diode_SMD:D_SOD-323_HandSoldering
- removed J3: Conn_01x12_Male, kicad-harwin:Harwin_M20-89012xx_1x12_P2.54mm_Horizontal
- removed SW15: SW_Push, custom:CherryMX_Choc_1u
- SW10: footprint custom:CherryMX_Choc_1u -> Button_Switch_Keyboard:SW_Cherry_MX_2.25u_PCB
- SW12, SW17, SW18, SW19, SW21, SW22, SW23, SW3, SW31, SW32, SW33, SW4, SW5, SW7, SW8, SW9: footprint custom:CherryMX_Choc_1u -> Button_Switch_Keyboard:SW_Cherry_MX_1.00u_PCB
- SW13, SW24, SW34: footprint custom:CherryMX_Choc_1u -> Button_Switch_Keyboard:SW_Cherry_MX_1.25u_PCB
- SW14: footprint custom:CherryMX_Choc_1u -> Button_Switch_Keyboard:SW_Cherry_MX_1.50u_PCB
- moved C2 240.4 mm to (-3.56, 33.0), turned to 270 degrees
- moved D14 238.1 mm to (-2.41, 59.9)
- moved D15 238.1 mm to (-2.41, 65.5)
- moved D33 234.1 mm to (-0.38, 59.9)
- moved D34 234.1 mm to (-0.38, 65.5)
- moved C3 232.1 mm to (6.10, 33.3)
- moved D12 230.2 mm to (-0.38, 75.6)
- moved D36 230.2 mm to (3.68, 75.6)
- moved D26 230.2 mm to (1.65, 75.6)
- moved U1 230.2 mm to (1.52, 39.1)
- moved D23 230.1 mm to (1.65, 59.9)
- moved D24 230.1 mm to (1.65, 65.5)
- moved R7 229.4 mm to (1.65, 26.4)
- moved R6 229.4 mm to (-2.92, 26.4)
- moved C5 229.3 mm to (-3.56, 45.7)
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Connections:
- J1 pad A8: Net-(J1-PadA8) -> (no net)
- J1 pad B8: Net-(J1-PadB8) -> (no net)
- J2 pad 3: TX -> RX
- J2 pad 4: RX -> TX
- SW10 pad 2: COL3 -> COL6
- SW12 pad 2: COL6 -> COL1
- SW13 pad 2: COL6 -> COL1
- SW14 pad 2: COL6 -> COL1
- SW17 pad 2: COL2 -> COL5
- SW18 pad 2: COL2 -> COL5
- SW19 pad 2: COL2 -> COL5
- SW21 pad 2: COL4 -> COL3
- SW22 pad 2: COL4 -> COL3
- SW23 pad 2: COL4 -> COL3
- SW24 pad 2: COL4 -> COL5
- SW3 pad 2: COL1 -> COL6
- SW31 pad 2: COL5 -> COL2
- SW32 pad 2: COL5 -> COL2
- SW33 pad 2: COL5 -> COL2
- SW34 pad 2: COL5 -> COL4
- SW4 pad 2: COL1 -> COL6
- SW5 pad 2: COL1 -> COL6
- SW7 pad 2: COL3 -> COL4
- SW8 pad 2: COL3 -> COL4
- SW9 pad 2: COL3 -> COL4
- U1 pad 1: VBAT -> (no net)
- U1 pad 10: Net-(U1-Pad10) -> (no net)
- U1 pad 11: Net-(U1-Pad11) -> (no net)
- U1 pad 12: Net-(U1-Pad12) -> (no net)
- U1 pad 13: Net-(U1-Pad13) -> (no net)
- U1 pad 14: PA4 -> (no net)
- U1 pad 15: PA5 -> (no net)
- U1 pad 16: PA6 -> (no net)
- U1 pad 17: PA7 -> (no net)
- U1 pad 2: Net-(U1-Pad2) -> (no net)
- U1 pad 22: Net-(U1-Pad22) -> (no net)
- U1 pad 25: GND -> 3.3V
- U1 pad 26: Net-(U1-Pad26) -> (no net)
- U1 pad 27: Net-(U1-Pad27) -> (no net)
- U1 pad 28: Net-(U1-Pad28) -> (no net)
- U1 pad 29: Net-(U1-Pad29) -> (no net)
- U1 pad 3: Net-(U1-Pad3) -> (no net)
- U1 pad 34: SWDIO -> (no net)
- U1 pad 37: SWDCLK -> (no net)
- U1 pad 38: COL1 -> COL6
- U1 pad 39: COL2 -> COL5
- U1 pad 4: Net-(U1-Pad4) -> (no net)
- U1 pad 40: COL3 -> COL4
- U1 pad 41: COL4 -> COL3
- U1 pad 42: PB6 -> (no net)
- U1 pad 43: PB7 -> (no net)
- U1 pad 45: COL5 -> COL2
- U1 pad 46: COL6 -> COL1
- U1 pad 5: Net-(U1-Pad5) -> (no net)
- U1 pad 6: Net-(U1-Pad6) -> (no net)
Routing:
- net COL6: track 96.7 -> 218.4 mm
- net COL1: track 182.5 -> 88.6 mm
- net COL5: track 122.1 -> 212.2 mm
- net COL2: track 162.9 -> 104.1 mm
- net COL4: track 143.4 -> 197.0 mm
- net COL3: track 164.9 -> 122.2 mm
- net Net-(D12-Pad2): track 73.7 -> 115.1 mm
- net SWDCLK: track 32.3 -> 0.00 mm, vias 1 -> 0
- net Net-(D7-Pad2): track 116.8 -> 148.9 mm
- net Net-(D21-Pad2): track 99.0 -> 130.6 mm
- net SWDIO: track 30.6 -> 0.00 mm, vias 1 -> 0
- net Net-(D11-Pad2): track 86.2 -> 111.6 mm
- net Net-(D26-Pad2): track 55.6 -> 78.9 mm
- net Net-(D17-Pad2): track 20.9 -> 0.00 mm
- net PB7: track 18.2 -> 0.00 mm, vias 1 -> 0
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Other:
- board size 135.9 x 89.9 mm -> 146.1 x 78.7 mm
- rule pad_to_mask_clearance: 0 -> 0.051
- board text added: "NotKeySeeBee v0.4 by NotTeXitoi"
- board text removed: "3.3V"
- board text removed: "5V"
- board text removed: "GND"
- board text removed: "KeySeeBee v0.2 by TeXitoi"
- board text removed: "PA4"
- board text removed: "PA5"
- board text removed: "PA6"
- board text removed: "PA7"
- board text removed: "PB6"
- board text removed: "PB7"
- board text removed: "SWDCLK"
- board text removed: "SWDIO"
